Commit message: Add Simplified Geometries Fingers

File: franka_description/robots/hand_original.xacro (robot description, xacro)
@@ -43,7 +43,7 @@
       </visual>
       <collision>
-        <origin xyz="0.0 0.0045 0.057" rpy="0 0 0"/>
+        <origin xyz="-0.0045 0.0045 0.05" rpy="${pi/2} ${pi} 0"/>
         <geometry>
-          <box size="0.018 0.009 0.04" />
+          <mesh filename="package://franka_description/meshes/collision/Finger_Robothon_3l.stl" scale="0.001 0.001 0.001"/>
         </geometry>
       </collision>
@@ -57,7 +57,7 @@
       </visual>
       <collision>
-        <origin xyz="0.0 -0.0045 0.057" rpy="0 0 0" />
+       <origin xyz="0.0045 -0.0045 0.05" rpy="${pi/2} ${pi} ${pi}"/>
         <geometry>
-          <box size="0.018 0.009 0.04" />
+          <mesh filename="package://franka_description/meshes/collision/Finger_Robothon_3r.stl" scale="0.001 0.001 0.001"/>
         </geometry>
       </collision>

File: franka_description/robots/hand_robothon.xacro (robot description, xacro)
@@ -43,7 +43,7 @@
       </visual>
       <collision>
-        <origin xyz="0.0 0.0045 0.057" rpy="0 0 0"/>
+        <origin xyz="0.0 0.0 0.05" rpy="0 0 0"/>
         <geometry>
-          <box size="0.018 0.009 0.04" />
+          <box size="0.02 0.01 0.04" />
         </geometry>
       </collision>
@@ -57,7 +57,7 @@
       </visual>
       <collision>
-        <origin xyz="0.0 -0.0045 0.057" rpy="0 0 0" />
+        <origin xyz="0.0 0.0 0.05" rpy="0 0 0" />
         <geometry>
-          <box size="0.018 0.009 0.04" />
+          <box size="0.02 0.01 0.04" />
         </geometry>
       </collision>

File: franka_description/robots/panda_arm.urdf.xacro (robot description, xacro)
@@ -8,8 +8,8 @@
     <!-- Create a URDF for a real hardware -->
     <xacro:include filename="$(find franka_description)/robots/panda_arm.xacro" />
-    <xacro:panda_arm arm_id="${arm_id}" safety_distance="0.03"/>
+    <xacro:panda_arm arm_id="${arm_id}" safety_distance="0.0"/>
     <xacro:if value="$(arg hand)">
       <xacro:include filename="$(find franka_description)/robots/hand.xacro"/>
-      <xacro:hand ns="${arm_id}" rpy="0 0 ${-pi/4}" connected_to="${arm_id}_link8" safety_distance="0.03"/>
+      <xacro:hand ns="${arm_id}" rpy="0 0 ${-pi/4}" connected_to="${arm_id}_link8" safety_distance="0.0"/>
     </xacro:if>
   </xacro:unless>
